File: MCP2221A_Board.kicad_sch (KiCad schematic)
At the start: 22 parts, among them J1 USB_B_Mini, J2 Conn_02x04_Odd_Even, SW1 I/O, U2 MCP2221AxSL, U3 LD1117S33TR_SOT223

Commit message: Updated documentation
Other:
- title: (none) -> MCP2221A Board
Changed lines of the file:
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@@
 	(generator_version "8.0")
 	(paper "A4")
+	(title_block
+		(title "MCP2221A Board")
+		(date "2024-09-18")
+		(rev "0.1")
+	)
 	(junction
 		(at 31.75 134.62)
